Commit message: Got the URDF file in order with the correct joints and components positions

File: roomba_robot/src/roombot/urdf/roombot_physical.urdf (robot description, URDF)
Before this commit: robot roomba_bot, 6 links, 5 joints
Links:
- removed link bno055
- added link imu_link
- link base_link: geometry collision cylinder length=0.0762 radius=0.1651; visual cylinder length=0.0762 radius=0.1651
- link left_wheel_link: mass 0.2 -> None; geometry collision cylinder length=0.026 radius=0.0331; visual cylinder length=0.026 radius=0.0331
- link lidar_link: mass 0.08 -> None; geometry collision cylinder length=0.05 radius=0.05; visual cylinder length=0.05 radius=0.05
- link right_wheel_link: mass 0.2 -> None; geometry collision cylinder length=0.026 radius=0.0331; visual cylinder length=0.026 radius=0.0331
Joints:
- removed joint bno055_joint
- added joint imu_joint: type fixed, parent base_link, child imu_link, origin xyz=0.056 0.075 0.05 rpy=0 0 0
- joint caster_joint: origin xyz=-0.090 0.000 0.000 rpy=0 0 0 -> xyz=0.127 0.000 -0.03 rpy=1.57 0 0
- joint left_wheel_joint: axis (none) -> 0 0 1; origin xyz=0.000 0.080 0.000 rpy=0 0 0 -> xyz=0 0.1143 -0.02 rpy=1.57 0 0; type fixed -> continuous
- joint lidar_joint: origin xyz=0.090 0.000 0.060 rpy=0 0 0 -> xyz=-0.08255 0.00635 0.0889 rpy=0 0 0
- joint right_wheel_joint: axis (none) -> 0 0 1; origin xyz=0.000 -0.080 0.000 rpy=0 0 0 -> xyz=0 -0.1143 -0.02 rpy=1.57 0 0; type fixed -> continuous
